File: gr65_matrix.kicad_sch (KiCad schematic)
At the start: 152 parts, among them SW1 SW_Push, SW10 SW_Push, SW11 SW_Push, SW12 SW_Push, SW13 SW_Push, SW14 SW_Push, SW15 SW_Push, SW16 SW_Push, SW17 SW_Push, SW18 SW_Push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

Commit message: Update matrix positions
Parts:
- renumbered SW29_0 to SW29_ANSI, SW43_1 to SW43_ISO, SW44_1 to SW44_ANSI, SW44_0 to SW44_ISO, SW46_1 to SW46_ANSI, SW46_0 to SW46_ISO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
Other:
- moved on the sheet: SW1, SW10, SW11, SW12, SW13, SW14, SW15, SW16, SW17, SW18, SW19, SW2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
