File: gr65_matrix.kicad_sch (KiCad schematic)
At the start: 152 parts, among them SW1 SW_Push, SW10 SW_Push, SW11 SW_Push, SW12 SW_Push, SW13 SW_Push, SW14 SW_Push, SW15 SW_Push, SW16 SW_Push, SW17 SW_Push, SW18 SW_Push, SW19 SW_Push, SW2 SW_Push, SW20 SW_Push, SW21 SW_Push, SW22 SW_Push, SW23 SW_Push, SW24 SW_Push, SW25 SW_Push, SW26 SW_Push, SW27 SW_Push, SW28 SW_Push, SW29_ANSI SW_Push, SW3 SW_Push, SW30 SW_Push, SW31 SW_Push, SW32 SW_Push, SW33 SW_Push, SW34 SW_Push, SW35 SW_Push, SW36 SW_Push, SW37 SW_Push, SW38 SW_Push, SW39 SW_Push, SW4 SW_Push, SW40 SW_Push, SW41 SW_Push, SW42 SW_Push, SW43_ISO SW_Push, SW44_ANSI SW_Push, SW44_ISO SW_Push, SW45 SW_Push, SW46_ANSI SW_Push, SW46_ISO SW_Push, SW47_ISO SW_Push, SW48 SW_Push, SW49 SW_Push, SW5 SW_Push, SW50 SW_Push, SW51 SW_Push, SW52 SW_Push, SW53 SW_Push, SW54 SW_Push, SW55 SW_Push, SW56 SW_Push, SW57 SW_Push, SW58 SW_Push, SW59 SW_Push, SW6 SW_Push, SW60 SW_Push, SW61 SW_Push, SW62 SW_Push, SW63 SW_Push, SW64 SW_Push, SW65 SW_Push, SW66 SW_Push, SW67 SW_Push, SW68 SW_Push, SW69 SW_Push, SW7 SW_Push, SW70 SW_Push, SW71 SW_Push, SW72 SW_Push, SW73 SW_Push, SW74 SW_Push, SW75 SW_Push, SW8 SW_Push, SW9 SW_Push

Commit message: Update pcb with exploded layout
Parts:
- removed SW44_ANSI: SW_Push, Switch_Keyboard_Hotswap_Kailh:SW_Hotswap_Kailh_MX_ISOEnter, symbol Switch:SW_Push
- removed SW46_ANSI: SW_Push, Switch_Keyboard_Hotswap_Kailh:SW_Hotswap_Kailh_MX_1.25u, symbol Switch:SW_Push
- D1, D10, D11, D12, D13, D14, D16, D17, D18, D19, D2, D20, D21, D22, D23, D24, D25, D26, D27, D28, D3, D31, D32, D33, D34, D35, D36, D37, D38, D39, D4, D40, D41, D42, D44, D46, D48, D49, D5, D50, D51, D52, D53, D54, D55, D56, D58, D59, D6, D60, D61, D62, D63, D7, D70, D71, D72, D73, D74, D75, D8, D9: footprint Diode_THT:D_DO-35_SOD27_P7.62mm_Horizontal -> Diode_SMD:D_SOD-123
- D15, D30, D43, D45, D47, SW15, SW30, SW45: now not fitted; now left out of the parts list
- D29: footprint Diode_THT:D_DO-35_SOD27_P7.62mm_Horizontal -> Diode_SMD:D_SOD-123; now left out of the parts list
- D57: footprint Diode_THT:D_DO-35_SOD27_P7.62mm_Horizontal -> Diode_SMD:D_SOD-123; now fitted; now in the parts list
- D67: footprint Diode_THT:D_DO-35_SOD27_P7.62mm_Horizontal -> Diode_SMD:D_SOD-123; now in the parts list
- SW29: renamed from SW29_ANSI; now left out of the parts list
- SW43: renamed from SW43_ISO; now not fitted; now left out of the parts list
- SW47: renamed from SW47_ISO; now not fitted; now left out of the parts list
- SW57: now fitted; now in the parts list
- SW67: now in the parts list
- renumbered SW44_ISO to SW44, SW46_ISO to SW46
Other:
- moved on the sheet: SW44, SW46
