File: gr65.kicad_pcb (KiCad board)
At the start: 2 copper layers, 151 parts, among them SW1 SW_Push, SW10 SW_Push, SW11 SW_Push, SW12 SW_Push, SW13 SW_Push, SW14 SW_Push, SW15 SW_Push, SW16 SW_Push, SW17 SW_Push, SW18 SW_Push, SW19 SW_Push, SW2 SW_Push, SW20 SW_Push, SW21 SW_Push, SW22 SW_Push, SW23 SW_Push, SW24 SW_Push, SW25 SW_Push, SW26 SW_Push, SW27 SW_Push, SW28 SW_Push, SW29 SW_Push, SW3 SW_Push, SW30 SW_Push, SW31 SW_Push, SW32 SW_Push, SW33 SW_Push, SW34 SW_Push, SW35 SW_Push, SW36 SW_Push, SW37 SW_Push, SW38 SW_Push, SW39 SW_Push, SW4 SW_Push, SW40 SW_Push, SW41 SW_Push, SW42 SW_Push, SW43 SW_Push, SW44 SW_Push, SW45 SW_Push, SW46 SW_Push, SW47 SW_Push, SW48 SW_Push, SW49 SW_Push, SW5 SW_Push, SW50 SW_Push, SW51 SW_Push, SW52 SW_Push, SW53 SW_Push, SW54 SW_Push, SW55 SW_Push, SW56 SW_Push, SW57 SW_Push, SW58 SW_Push, SW59 SW_Push, SW6 SW_Push, SW60 SW_Push, SW61 SW_Push, SW62 SW_Push, SW63 SW_Push, SW64 SW_Push, SW65 SW_Push, SW66 SW_Push, SW67 SW_Push, SW68 SW_Push, SW69 SW_Push, SW7 SW_Push, SW70 SW_Push, SW71 SW_Push, SW72 SW_Push, SW73 SW_Push, SW74 SW_Push, SW75 SW_Push, SW8 SW_Push, SW9 SW_Push

Commit message: Update pcb with exploded layout
Parts:
- removed D15, D30, D43, D45, D47, D64, D65, D66, D68, D69: 1N4148, Diode_THT:D_DO-35_SOD27_P7.62mm_Horizontal
- removed SW15, SW30, SW43, SW45, SW47, SW64, SW65, SW66, SW69: SW_Push, Switch_Keyboard_Hotswap_Kailh:SW_Hotswap_Kailh_MX_1.00u
- removed SW68: SW_Push, Switch_Keyboard_Hotswap_Kailh:SW_Hotswap_Kailh_MX_6.25u
- added S14: Stabilizer_Cherry_MX_2.00u, Mounting_Keyboard_Stabilizer:Stabilizer_Cherry_MX_2.00u, F.Cu at (319.1, 109.5)
- added S44: Stabilizer_Cherry_MX_2.00u, Mounting_Keyboard_Stabilizer:Stabilizer_Cherry_MX_2.00u, F.Cu at (316.7, 147.6)
- added S46: Stabilizer_Cherry_MX_2.00u, Mounting_Keyboard_Stabilizer:Stabilizer_Cherry_MX_2.00u, F.Cu at (73.8, 166.7)
- added S67: Stabilizer_Cherry_MX_6.25u, Mounting_Keyboard_Stabilizer:Stabilizer_Cherry_MX_6.25u, F.Cu at (183.4, 185.7)
- D1, D10, D11, D12, D13, D14, D16, D17, D18, D19, D2, D20, D21, D22, D23, D24, D25, D26, D27, D28, D29, D3, D31, D32, D33, D34, D35, D36, D37, D38, D39, D4, D40, D41, D42, D44, D46, D48, D49, D5, D50, D51, D52, D53, D54, D55, D56, D57, D58, D59, D6, D60, D61, D62, D63, D67, D7, D70, D71, D72, D73, D74, D75, D8, D9: footprint Diode_THT:D_DO-35_SOD27_P7.62mm_Horizontal -> Diode_SMD:D_SOD-123; moved to B.Cu
- SW67: footprint Switch_Keyboard_Hotswap_Kailh:SW_Hotswap_Kailh_MX_1.00u -> Switch_Keyboard_Hotswap_Kailh:SW_Hotswap_Kailh_MX_6.25u
- moved SW14 260.4 mm to (319.1, 109.5)
- moved SW29 248.3 mm to (323.9, 128.6)
- moved SW13 234.6 mm to (290.5, 109.5)
- moved SW60 230.2 mm to (357.2, 166.7)
- moved SW28 223.3 mm to (300.0, 128.6)
- moved SW12 219.8 mm to (271.5, 109.5)
- moved SW44 217.5 mm to (316.7, 147.6)
- moved SW75 214.8 mm to (352.4, 190.5)
- moved SW11 206.9 mm to (252.4, 109.5)
- moved SW59 206.9 mm to (333.4, 171.5)
- moved SW74 205.9 mm to (333.4, 190.5)
- moved SW27 203.9 mm to (281.0, 128.6)
- moved SW42 201.8 mm to (285.8, 147.6)
- moved SW73 199.7 mm to (314.3, 190.5)
- moved SW10 199.6 mm to (233.4, 109.5)
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Connections:
- net COL0 renamed /COL0
- net COL1 renamed /COL1
- net COL10 renamed /COL10
- net COL11 renamed /COL11
- net COL12 renamed /COL12
- net COL13 renamed /COL13
- net COL14 renamed /COL14
- net COL2 renamed /COL2
- net COL3 renamed /COL3
- net COL4 renamed /COL4
- net COL5 renamed /COL5
- net COL6 renamed /COL6
- net COL7 renamed /COL7
- net COL8 renamed /COL8
- net COL9 renamed /COL9
- net ROW0 renamed /ROW0
- net ROW1 renamed /ROW1
- net ROW2 renamed /ROW2
- net ROW3 renamed /ROW3
- net ROW4 renamed /ROW4
Routing:
- net /ROW3: track 0.00 -> 424.2 mm, vias 0 -> 14
- net /ROW0: track 0.00 -> 394.1 mm, vias 0 -> 15
- net /ROW1: track 0.00 -> 393.1 mm, vias 0 -> 15
- net /ROW4: track 0.00 -> 390.5 mm, vias 0 -> 10
- net /ROW2: track 0.00 -> 374.9 mm, vias 0 -> 13
- net /COL0: track 0.00 -> 96.8 mm
- net Net-(D3-A): track 0.00 -> 16.0 mm
- net Net-(D41-A): track 0.00 -> 16.0 mm
- net Net-(D1-A): track 0.00 -> 16.0 mm
- net Net-(D2-A): track 0.00 -> 16.0 mm
- net Net-(D16-A): track 0.00 -> 16.0 mm
- net Net-(D4-A): track 0.00 -> 16.0 mm
- net Net-(D17-A): track 0.00 -> 16.0 mm
- net Net-(D5-A): track 0.00 -> 16.0 mm
- net Net-(D18-A): track 0.00 -> 16.0 mm
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Other:
- board outline added: 314.3 x 100 mm
