File: hzk65_matrix.kicad_sch (KiCad schematic)
At the start: 150 parts, among them SW1 SW_Push, SW10 SW_Push, SW11 SW_Push, SW12 SW_Push, SW13 SW_Push, SW14 SW_Push, SW15 SW_Push, SW16 SW_Push, SW17 SW_Push, SW18 SW_Push, SW19 SW_Push, SW2 SW_Push, SW20 SW_Push, SW21 SW_Push, SW22 SW_Push, SW23 SW_Push, SW24 SW_Push, SW25 SW_Push, SW26 SW_Push, SW27 SW_Push, SW28 SW_Push, SW29 SW_Push, SW3 SW_Push, SW30 SW_Push, SW31 SW_Push, SW32 SW_Push, SW33 SW_Push, SW34 SW_Push, SW35 SW_Push, SW36 SW_Push, SW37 SW_Push, SW38 SW_Push, SW39 SW_Push, SW4 SW_Push, SW40 SW_Push, SW41 SW_Push, SW42 SW_Push, SW43 SW_Push, SW44 SW_Push, SW45 SW_Push, SW46 SW_Push, SW47 SW_Push, SW48 SW_Push, SW49 SW_Push, SW5 SW_Push, SW50 SW_Push, SW51 SW_Push, SW52 SW_Push, SW53 SW_Push, SW54 SW_Push, SW55 SW_Push, SW56 SW_Push, SW57 SW_Push, SW58 SW_Push, SW59 SW_Push, SW6 SW_Push, SW60 SW_Push, SW61 SW_Push, SW62 SW_Push, SW63 SW_Push, SW64 SW_Push, SW65 SW_Push, SW66 SW_Push, SW67 SW_Push, SW68 SW_Push, SW69 SW_Push, SW7 SW_Push, SW70 SW_Push, SW71 SW_Push, SW72 SW_Push, SW73 SW_Push, SW74 SW_Push, SW75 SW_Push, SW8 SW_Push, SW9 SW_Push

Commit message: Update key matrix disposition
Parts:
- D29, SW29: now in the parts list
- SW15, SW30, SW43, SW45, SW47, SW64, SW65, SW66, SW68, SW69: footprint Switch_Keyboard_Hotswap_Kailh:SW_Hotswap_Kailh_MX_1.00u -> (none)
Connections:
- net COL0: now also SW1.2, SW16.2, SW31.2, SW46.2, SW61.2; no longer D1.1 (K), D16.1 (K), D31.1 (K), D46.1 (K), D61.1 (K)
- net COL1: now also SW17.2, SW2.2, SW32.2, SW47.2, SW62.2; no longer D17.1 (K), D2.1 (K), D32.1 (K), D47.1 (K), D62.1 (K)
- net COL10: now also SW11.2, SW26.2, SW41.2, SW56.2, SW71.2; no longer D11.1 (K), D26.1 (K), D41.1 (K), D56.1 (K), D71.1 (K)
- net COL11: now also SW12.2, SW27.2, SW42.2, SW57.2, SW72.2; no longer D12.1 (K), D27.1 (K), D42.1 (K), D57.1 (K), D72.1 (K)
- net COL12: now also SW13.2, SW28.2, SW43.2, SW58.2, SW73.2; no longer D13.1 (K), D28.1 (K), D43.1 (K), D58.1 (K), D73.1 (K)
- net COL13: now also SW14.2, SW29.2, SW44.2, SW59.2, SW74.2; no longer D14.1 (K), D29.1 (K), D44.1 (K), D59.1 (K), D74.1 (K)
- net COL14: now also SW15.2, SW30.2, SW45.2, SW60.2, SW75.2; no longer D15.1 (K), D30.1 (K), D45.1 (K), D60.1 (K), D75.1 (K)
- net COL2: now also SW18.2, SW3.2, SW33.2, SW48.2, SW63.2; no longer D18.1 (K), D3.1 (K), D33.1 (K), D48.1 (K), D63.1 (K)
- net COL3: now also SW19.2, SW34.2, SW4.2, SW49.2, SW64.2; no longer D19.1 (K), D34.1 (K), D4.1 (K), D49.1 (K), D64.1 (K)
- net COL4: now also SW20.2, SW35.2, SW5.2, SW50.2, SW65.2; no longer D20.1 (K), D35.1 (K), D5.1 (K), D50.1 (K), D65.1 (K)
- net COL5: now also SW21.2, SW36.2, SW51.2, SW6.2, SW66.2; no longer D21.1 (K), D36.1 (K), D51.1 (K), D6.1 (K), D66.1 (K)
- net COL6: now also SW22.2, SW37.2, SW52.2, SW67.2, SW7.2; no longer D22.1 (K), D37.1 (K), D52.1 (K), D67.1 (K), D7.1 (K)
- net COL7: now also SW23.2, SW38.2, SW53.2, SW68.2, SW8.2; no longer D23.1 (K), D38.1 (K), D53.1 (K), D68.1 (K), D8.1 (K)
- net COL8: now also SW24.2, SW39.2, SW54.2, SW69.2, SW9.2; no longer D24.1 (K), D39.1 (K), D54.1 (K), D69.1 (K), D9.1 (K)
- net COL9: now also SW10.2, SW25.2, SW40.2, SW55.2, SW70.2; no longer D10.1 (K), D25.1 (K), D40.1 (K), D55.1 (K), D70.1 (K)
- net ROW0: now also D1.2 (A), D10.2 (A), D11.2 (A), D12.2 (A), D13.2 (A), D14.2 (A), D15.2 (A), D2.2 (A), D3.2 (A), D4.2 (A), D5.2 (A), D6.2 (A), D7.2 (A), D8.2 (A), D9.2 (A); no longer SW1.1, SW10.1, SW11.1, SW12.1, SW13.1, SW14.1, SW15.1, SW2.1, SW3.1, SW4.1, SW5.1, SW6.1, SW7.1, SW8.1, SW9.1
- net ROW1: now also D16.2 (A), D17.2 (A), D18.2 (A), D19.2 (A), D20.2 (A), D21.2 (A), D22.2 (A), D23.2 (A), D24.2 (A), D25.2 (A), D26.2 (A), D27.2 (A), D28.2 (A), D29.2 (A), D30.2 (A); no longer SW16.1, SW17.1, SW18.1, SW19.1, SW20.1, SW21.1, SW22.1, SW23.1, SW24.1, SW25.1, SW26.1, SW27.1, SW28.1, SW29.1, SW30.1
- net ROW2: now also D31.2 (A), D32.2 (A), D33.2 (A), D34.2 (A), D35.2 (A), D36.2 (A), D37.2 (A), D38.2 (A), D39.2 (A), D40.2 (A), D41.2 (A), D42.2 (A), D43.2 (A), D44.2 (A), D45.2 (A); no longer SW31.1, SW32.1, SW33.1, SW34.1, SW35.1, SW36.1, SW37.1, SW38.1, SW39.1, SW40.1, SW41.1, SW42.1, SW43.1, SW44.1, SW45.1
- net ROW3: now also D46.2 (A), D47.2 (A), D48.2 (A), D49.2 (A), D50.2 (A), D51.2 (A), D52.2 (A), D53.2 (A), D54.2 (A), D55.2 (A), D56.2 (A), D57.2 (A), D58.2 (A), D59.2 (A), D60.2 (A); no longer SW46.1, SW47.1, SW48.1, SW49.1, SW50.1, SW51.1, SW52.1, SW53.1, SW54.1, SW55.1, SW56.1, SW57.1, SW58.1, SW59.1, SW60.1
- net ROW4: now also D61.2 (A), D62.2 (A), D63.2 (A), D64.2 (A), D65.2 (A), D66.2 (A), D67.2 (A), D68.2 (A), D69.2 (A), D70.2 (A), D71.2 (A), D72.2 (A), D73.2 (A), D74.2 (A), D75.2 (A); no longer SW61.1, SW62.1, SW63.1, SW64.1, SW65.1, SW66.1, SW67.1, SW68.1, SW69.1, SW70.1, SW71.1, SW72.1, SW73.1, SW74.1, SW75.1
- new net: D44.1 (K), SW44.1
- new net: D22.1 (K), SW22.1
- new net: D49.1 (K), SW49.1
- new net: D62.1 (K), SW62.1
- new net: D3.1 (K), SW3.1
- new net: D20.1 (K), SW20.1
- new net: D10.1 (K), SW10.1
- new net: D52.1 (K), SW52.1
- new net: D59.1 (K), SW59.1
- new net: D53.1 (K), SW53.1
- new net: D23.1 (K), SW23.1
- new net: D33.1 (K), SW33.1
- new net: D47.1 (K), SW47.1
- new net: D21.1 (K), SW21.1
- new net: D15.1 (K), SW15.1
- new net: D34.1 (K), SW34.1
- new net: D36.1 (K), SW36.1
- new net: D57.1 (K), SW57.1
- new net: D51.1 (K), SW51.1
- new net: D75.1 (K), SW75.1
- new net: D55.1 (K), SW55.1
- new net: D4.1 (K), SW4.1
- new net: D41.1 (K), SW41.1
- new net: D1.1 (K), SW1.1
- new net: D11.1 (K), SW11.1
- new net: D27.1 (K), SW27.1
- new net: D17.1 (K), SW17.1
- new net: D6.1 (K), SW6.1
- new net: D18.1 (K), SW18.1
- new net: D37.1 (K), SW37.1
- new net: D7.1 (K), SW7.1
- new net: D50.1 (K), SW50.1
- new net: D42.1 (K), SW42.1
- new net: D73.1 (K), SW73.1
- new net: D31.1 (K), SW31.1
- new net: D5.1 (K), SW5.1
- new net: D45.1 (K), SW45.1
- new net: D67.1 (K), SW67.1
- new net: D65.1 (K), SW65.1
- new net: D60.1 (K), SW60.1
- new net: D72.1 (K), SW72.1
- new net: D46.1 (K), SW46.1
- new net: D43.1 (K), SW43.1
- new net: D29.1 (K), SW29.1
- new net: D8.1 (K), SW8.1
- new net: D66.1 (K), SW66.1
- new net: D13.1 (K), SW13.1
- new net: D2.1 (K), SW2.1
- new net: D24.1 (K), SW24.1
- new net: D63.1 (K), SW63.1
- new net: D26.1 (K), SW26.1
- new net: D61.1 (K), SW61.1
- new net: D70.1 (K), SW70.1
- new net: D30.1 (K), SW30.1
- new net: D68.1 (K), SW68.1
- new net: D69.1 (K), SW69.1
- new net: D64.1 (K), SW64.1
- new net: D48.1 (K), SW48.1
- new net: D39.1 (K), SW39.1
- new net: D14.1 (K), SW14.1
- new net: D58.1 (K), SW58.1
- new net: D35.1 (K), SW35.1
- new net: D16.1 (K), SW16.1
- new net: D54.1 (K), SW54.1
- new net: D19.1 (K), SW19.1
- new net: D38.1 (K), SW38.1
- new net: D40.1 (K), SW40.1
- new net: D56.1 (K), SW56.1
- new net: D32.1 (K), SW32.1
- new net: D71.1 (K), SW71.1
- new net: D74.1 (K), SW74.1
- new net: D25.1 (K), SW25.1
- new net: D9.1 (K), SW9.1
- new net: D12.1 (K), SW12.1
- new net: D28.1 (K), SW28.1
