File: hzk65.kicad_pcb (KiCad board)
At the start: 2 copper layers, 314.3 x 100 mm, 136 parts, among them SW1 SW_Push, SW10 SW_Push, SW11 SW_Push, SW12 SW_Push, SW13 SW_Push, SW14 SW_Push, SW16 SW_Push, SW17 SW_Push, SW18 SW_Push, SW19 SW_Push, SW2 SW_Push, SW20 SW_Push, SW21 SW_Push, SW22 SW_Push, SW23 SW_Push, SW24 SW_Push, SW25 SW_Push, SW26 SW_Push, SW27 SW_Push, SW28 SW_Push, SW29 SW_Push, SW3 SW_Push, SW31 SW_Push, SW32 SW_Push, SW33 SW_Push, SW34 SW_Push, SW35 SW_Push, SW36 SW_Push, SW37 SW_Push, SW38 SW_Push, SW39 SW_Push, SW4 SW_Push, SW40 SW_Push, SW41 SW_Push, SW42 SW_Push, SW44 SW_Push, SW46 SW_Push, SW48 SW_Push, SW49 SW_Push, SW5 SW_Push, SW50 SW_Push, SW51 SW_Push, SW52 SW_Push, SW53 SW_Push, SW54 SW_Push, SW55 SW_Push, SW56 SW_Push, SW57 SW_Push, SW58 SW_Push, SW59 SW_Push, SW6 SW_Push, SW60 SW_Push, SW61 SW_Push, SW62 SW_Push, SW63 SW_Push, SW67 SW_Push, SW7 SW_Push, SW70 SW_Push, SW71 SW_Push, SW72 SW_Push, SW73 SW_Push, SW74 SW_Push, SW75 SW_Push, SW8 SW_Push, SW9 SW_Push

Commit message: Handle drc exclusions
Parts:
- moved GL1 0.60 mm to (60.7, 192.9)
Other:
- outline, holes or cut-outs redrawn
Changed lines of the file:
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@@
 	(footprint "Symbol:OSHW-Logo_7.5x8mm_SilkScreen"
 		(layer "F.Cu")
-		(at 61.3181 192.8814)
+		(at 60.722975 192.8814)
 		(descr "Open Source Hardware Logo")
 		(tags "Logo OSHW")
@@
 		)
 	)
-	(gr_poly
-		(pts
-			(xy 97.592011 109.540973) (xy 97.592011 151.015573) (xy 143.942725 151.015573) (xy 143.942725 164.018729)
-			(xy 97.592017 164.018729) (xy 97.592017 186.076195) (xy 97.558599 188.033408) (xy 97.458307 189.938391)
-			(xy 97.291086 191.79107) (xy 97.056879 193.59137) (xy 96.75563 195.339219) (xy 96.387283 197.034541)
-			(xy 95.951781 198.677263) (xy 95.449069 200.26731) (xy 94.879091 201.804607) (xy 94.241789 203.289082)
-			(xy 93.537108 204.720659) (xy 92.764992 206.099264) (xy 91.925385 207.424824) (xy 91.01823 208.697264)
-			(xy 90.043471 209.916509) (xy 89.001052 211.082487) (xy 87.904453 212.18106) (xy 86.757577 213.20837)
-			(xy 85.560501 214.164468) (xy 84.313304 215.049409) (xy 83.016062 215.863246) (xy 81.668854 216.606033)
-			(xy 80.271757 217.277824) (xy 78.824849 217.878672) (xy 77.328206 218.408632) (xy 75.781907 218.867755)
-			(xy 74.186029 219.256098) (xy 72.540651 219.573712) (xy 70.845848 219.820652) (xy 69.101699 219.996971)
-			(xy 67.308282 220.102723) (xy 65.465674 220.137962) (xy 63.623151 220.102721) (xy 61.829976 219.996964)
-			(xy 60.086203 219.820636) (xy 58.391887 219.573687) (xy 56.747084 219.256062) (xy 55.151849 218.867708)
-			(xy 53.606237 218.408574) (xy 52.110303 217.878605) (xy 50.664103 217.27775) (xy 49.267691 216.605955)
-			(xy 47.921123 215.863167) (xy 46.624454 215.049333) (xy 45.377739 214.164401) (xy 44.181032 213.208318)
-			(xy 43.034391 212.181031) (xy 41.937868 211.082487) (xy 40.895429 209.916503) (xy 39.920655 208.69724)
-			(xy 39.01349 207.424775) (xy 38.173876 206.099183) (xy 37.401757 204.720543) (xy 36.697076 203.28893)
-			(xy 36.059777 201.804421) (xy 35.489803 200.267093) (xy 34.987097 198.677023) (xy 34.551602 197.034288)
-			(xy 34.183262 195.338963) (xy 33.882021 193.591127) (xy 33.64782 191.790855) (xy 33.480604 189.938225)
-			(xy 33.380316 188.033313) (xy 33.3469 186.076195) (xy 33.34692 186.07502) (xy 48.053695 186.07502)
-			(xy 48.071694 187.393759) (xy 48.125729 188.679311) (xy 48.215855 189.930699) (xy 48.342129 191.146945)
-			(xy 48.504607 192.327073) (xy 48.703344 193.470105) (xy 48.938397 194.575064) (xy 49.209822 195.640974)
-			(xy 49.517674 196.666856) (xy 49.86201 197.651734) (xy 50.242886 198.594631) (xy 50.660358 199.494568)
-			(xy 51.114481 200.350571) (xy 51.605313 201.16166) (xy 52.132908 201.926859) (xy 52.697323 202.645191)
-			(xy 53.289796 203.312378) (xy 53.91101 203.936178) (xy 54.56068 204.516638) (xy 55.238523 205.053806)
-			(xy 55.944257 205.547729) (xy 56.677598 205.998455) (xy 57.438262 206.40603) (xy 58.225967 206.770502)
-			(xy 59.040429 207.091917) (xy 59.881365 207.370324) (xy 60.748491 207.60577) (xy 61.641525 207.798301)
-			(xy 62.560183 207.947965) (xy 63.504182 208.05481) (xy 64.473239 208.118882) (xy 65.46707 208.140229)
-			(xy 66.460923 208.118881) (xy 67.430166 208.054805) (xy 68.374492 207.947955) (xy 69.293597 207.798283)
-			(xy 70.187174 207.605744) (xy 71.054918 207.370291) (xy 71.896525 207.091877) (xy 72.711688 206.770454)
-			(xy 73.500102 206.405978) (xy 74.261462 205.9984) (xy 74.995462 205.547674) (xy 75.701797 205.053753)
-			(xy 76.380162 204.516591) (xy 77.03025 203.936141) (xy 77.651757 203.312357) (xy 78.244377 202.645191)
-			(xy 78.808773 201.926859) (xy 79.336354 201.16166) (xy 79.827176 200.350571) (xy 80.281293 199.494568)
-			(xy 80.698762 198.594631) (xy 81.079638 197.651734) (xy 81.423977 196.666856) (xy 81.731834 195.640974)
-			(xy 82.003264 194.575064) (xy 82.238324 193.470105) (xy 82.437068 192.327073) (xy 82.599552 191.146945)
-			(xy 82.725832 189.930699) (xy 82.815964 188.679311) (xy 82.870002 187.393759) (xy 82.888002 186.07502)
-			(xy 82.888002 164.018136) (xy 65.466251 164.018136) (xy 65.46707 164.017386) (xy 64.473299 164.038734)
-			(xy 63.504296 164.10281) (xy 62.560342 164.20966) (xy 61.641721 164.359331) (xy 60.748715 164.55187)
-			(xy 59.881609 164.787323) (xy 59.040686 165.065737) (xy 58.226228 165.387159) (xy 57.43852 165.751636)
-			(xy 56.677843 166.159214) (xy 55.944482 166.609941) (xy 55.23872 167.103862) (xy 54.56084 167.641025)
-			(xy 53.911125 168.221476) (xy 53.289858 168.845262) (xy 52.697323 169.512429) (xy 52.132927 170.23077)
-			(xy 51.605347 170.995799) (xy 51.114525 171.806562) (xy 50.660408 172.662108) (xy 50.242939 173.561484)
-			(xy 49.862062 174.503738) (xy 49.517723 175.487917) (xy 49.209866 176.513069) (xy 48.938435 177.578242)
-			(xy 48.703375 178.682482) (xy 48.504631 179.824839) (xy 48.342146 181.004358) (xy 48.215865 182.220089)
-			(xy 48.125734 183.471077) (xy 48.071696 184.756372) (xy 48.053695 186.07502) (xy 33.34692 186.07502)
-			(xy 33.380318 184.119067) (xy 33.480609 182.214323) (xy 33.64783 180.362017) (xy 33.882037 178.562199)
-			(xy 34.183286 176.814922) (xy 34.551633 175.120239) (xy 34.987135 173.4782) (xy 35.489847 171.888858)
-			(xy 36.059826 170.352266) (xy 36.697128 168.868474) (xy 37.401809 167.437536) (xy 38.173925 166.059503)
-			(xy 39.013533 164.734427) (xy 39.920689 163.46236) (xy 40.895449 162.243355) (xy 41.937868 161.077462)
-			(xy 43.034381 159.978889) (xy 44.181016 158.951581) (xy 45.377717 157.995483) (xy 46.624429 157.110543)
-			(xy 47.921098 156.296706) (xy 49.267666 155.553918) (xy 50.664079 154.882127) (xy 52.110282 154.281279)
-			(xy 53.606219 153.751319) (xy 55.151834 153.292195) (xy 56.747073 152.903852) (xy 58.391879 152.586238)
-			(xy 60.086198 152.339298) (xy 61.829973 152.162978) (xy 63.623151 152.057226) (xy 65.465674 152.021987)
-			(xy 82.887425 152.021987) (xy 82.887425 121.613372) (xy 61.9138 121.613372) (xy 61.9138 109.5398)
+	(gr_arc
+		(start 52.3873 102.39355)
+		(mid 53.084767 100.709767)
+		(end 54.76855 100.0123)
+		(stroke
+			(width 0.05)
+			(type default)
+		)
+		(layer "Edge.Cuts")
+	)
+	(gr_line
+		(start 52.3873 197.64795)
+		(end 52.3873 102.39355)
+		(stroke
+			(width 0.05)
+			(type default)
+		)
+		(layer "Edge.Cuts")
+	)
+	(gr_line
+		(start 54.76855 100.0123)
+		(end 364.337649 100.0123)
+		(stroke
+			(width 0.05)
+			(type default)
+		)
+		(layer "Edge.Cuts")
+	)
+	(gr_arc
+		(start 54.76855 200.0292)
+		(mid 53.084752 199.331748)
+		(end 52.3873 197.64795)
+		(stroke
+			(width 0.05)
+			(type default)
 		)
+		(layer "Edge.Cuts")
+	)
+	(gr_arc
+		(start 364.337649 100.0123)
+		(mid 366.021447 100.709752)
+		(end 366.718899 102.39355)
 		(stroke
-			(width 0)
-			(type solid)
+			(width 0.05)
+			(type default)
 		)
-		(fill yes)
-		(layer "F.SilkS")
+		(layer "Edge.Cuts")
+	)
+	(gr_line
+		(start 364.337649 200.0292)
+		(end 54.76855 200.0292)
+		(stroke
+			(width 0.05)
+			(type default)
+		)
+		(layer "Edge.Cuts")
+	)
+	(gr_line
+		(start 366.718899 102.39355)
+		(end 366.718899 197.64795)
+		(stroke
+			(width 0.05)
+			(type default)
+		)
+		(layer "Edge.Cuts")
 	)
-	(gr_rect
-		(start 52.3873 100.0123)
-		(end 366.718899 200.0292)
+	(gr_arc
+		(start 366.718899 197.64795)
+		(mid 366.021447 199.331748)
+		(end 364.337649 200.0292)
 		(stroke
 			(width 0.05)
 			(type default)
 		)
-		(fill no)
 		(layer "Edge.Cuts")
 	)

Commit message: Update stitching via grid
Routing:
- net Net-(D75-A): vias 1 -> 0
- net GND: vias 45 -> 160
- net /COL9: vias 3 -> 0
- net /COL8: vias 2 -> 0
- net /COL7: vias 2 -> 0
- net /COL6: vias 2 -> 0
- net /COL5: vias 2 -> 0
- net /COL4: vias 2 -> 0
- net /COL3: vias 2 -> 0
- net /COL2: vias 3 -> 0
- net /COL13: vias 2 -> 0
- net /COL12: vias 1 -> 0
- net /COL11: vias 3 -> 0
- net /COL10: vias 3 -> 0
- net /COL1: vias 2 -> 0
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
Commit message: Use bus routing for rows and cols
Parts:
- removed GL1: OSHW-Logo_7.5x8mm_SilkScreen, Symbol:OSHW-Logo_7.5x8mm_SilkScreen
Connections:
- D1 pad 1: /COL0 -> Net-(D1-K)
- D1 pad 2: Net-(D1-A) -> /ROW0
- D10 pad 1: /COL9 -> Net-(D10-K)
- D10 pad 2: Net-(D10-A) -> /ROW0
- D11 pad 1: /COL10 -> Net-(D11-K)
- D11 pad 2: Net-(D11-A) -> /ROW0
- D12 pad 1: /COL11 -> Net-(D12-K)
- D12 pad 2: Net-(D12-A) -> /ROW0
- D13 pad 1: /COL12 -> Net-(D13-K)
- D13 pad 2: Net-(D13-A) -> /ROW0
- D14 pad 1: /COL13 -> Net-(D14-K)
- D14 pad 2: Net-(D14-A) -> /ROW0
- D16 pad 1: /COL0 -> Net-(D16-K)
- D16 pad 2: Net-(D16-A) -> /ROW1
- D17 pad 1: /COL1 -> Net-(D17-K)
- D17 pad 2: Net-(D17-A) -> /ROW1
- D18 pad 1: /COL2 -> Net-(D18-K)
- D18 pad 2: Net-(D18-A) -> /ROW1
- D19 pad 1: /COL3 -> Net-(D19-K)
- D19 pad 2: Net-(D19-A) -> /ROW1
- D2 pad 1: /COL1 -> Net-(D2-K)
- D2 pad 2: Net-(D2-A) -> /ROW0
- D20 pad 1: /COL4 -> Net-(D20-K)
- D20 pad 2: Net-(D20-A) -> /ROW1
- D21 pad 1: /COL5 -> Net-(D21-K)
- D21 pad 2: Net-(D21-A) -> /ROW1
- D22 pad 1: /COL6 -> Net-(D22-K)
- D22 pad 2: Net-(D22-A) -> /ROW1
- D23 pad 1: /COL7 -> Net-(D23-K)
- D23 pad 2: Net-(D23-A) -> /ROW1
- D24 pad 1: /COL8 -> Net-(D24-K)
- D24 pad 2: Net-(D24-A) -> /ROW1
- D25 pad 1: /COL9 -> Net-(D25-K)
- D25 pad 2: Net-(D25-A) -> /ROW1
- D26 pad 1: /COL10 -> Net-(D26-K)
- D26 pad 2: Net-(D26-A) -> /ROW1
- D27 pad 1: /COL11 -> Net-(D27-K)
- D27 pad 2: Net-(D27-A) -> /ROW1
- D28 pad 1: /COL12 -> Net-(D28-K)
- D28 pad 2: Net-(D28-A) -> /ROW1
- D29 pad 1: /COL13 -> Net-(D29-K)
- D29 pad 2: Net-(D29-A) -> /ROW1
- D3 pad 1: /COL2 -> Net-(D3-K)
- D3 pad 2: Net-(D3-A) -> /ROW0
- D31 pad 1: /COL0 -> Net-(D31-K)
- D31 pad 2: Net-(D31-A) -> /ROW2
- D32 pad 1: /COL1 -> Net-(D32-K)
- D32 pad 2: Net-(D32-A) -> /ROW2
- D33 pad 1: /COL2 -> Net-(D33-K)
- D33 pad 2: Net-(D33-A) -> /ROW2
- D34 pad 1: /COL3 -> Net-(D34-K)
- D34 pad 2: Net-(D34-A) -> /ROW2
- D35 pad 1: /COL4 -> Net-(D35-K)
- D35 pad 2: Net-(D35-A) -> /ROW2
- D36 pad 1: /COL5 -> Net-(D36-K)
- D36 pad 2: Net-(D36-A) -> /ROW2
- D37 pad 1: /COL6 -> Net-(D37-K)
- D37 pad 2: Net-(D37-A) -> /ROW2
- D38 pad 1: /COL7 -> Net-(D38-K)
- D38 pad 2: Net-(D38-A) -> /ROW2
- D39 pad 1: /COL8 -> Net-(D39-K)
- D39 pad 2: Net-(D39-A) -> /ROW2
- D4 pad 1: /COL3 -> Net-(D4-K)
- D4 pad 2: Net-(D4-A) -> /ROW0
- D40 pad 1: /COL9 -> Net-(D40-K)
- D40 pad 2: Net-(D40-A) -> /ROW2
- D41 pad 1: /COL10 -> Net-(D41-K)
- D41 pad 2: Net-(D41-A) -> /ROW2
- D42 pad 1: /COL11 -> Net-(D42-K)
- D42 pad 2: Net-(D42-A) -> /ROW2
- D44 pad 1: /COL13 -> Net-(D44-K)
- D44 pad 2: Net-(D44-A) -> /ROW2
- D46 pad 1: /COL0 -> Net-(D46-K)
- D46 pad 2: Net-(D46-A) -> /ROW3
- D48 pad 1: /COL2 -> Net-(D48-K)
- D48 pad 2: Net-(D48-A) -> /ROW3
- D49 pad 1: /COL3 -> Net-(D49-K)
- D49 pad 2: Net-(D49-A) -> /ROW3
- D5 pad 1: /COL4 -> Net-(D5-K)
- D5 pad 2: Net-(D5-A) -> /ROW0
- D50 pad 1: /COL4 -> Net-(D50-K)
- D50 pad 2: Net-(D50-A) -> /ROW3
- D51 pad 1: /COL5 -> Net-(D51-K)
- D51 pad 2: Net-(D51-A) -> /ROW3
- D52 pad 1: /COL6 -> Net-(D52-K)
- D52 pad 2: Net-(D52-A) -> /ROW3
- D53 pad 1: /COL7 -> Net-(D53-K)
- D53 pad 2: Net-(D53-A) -> /ROW3
- D54 pad 1: /COL8 -> Net-(D54-K)
- D54 pad 2: Net-(D54-A) -> /ROW3
- D55 pad 1: /COL9 -> Net-(D55-K)
- D55 pad 2: Net-(D55-A) -> /ROW3
- D56 pad 1: /COL10 -> Net-(D56-K)
- D56 pad 2: Net-(D56-A) -> /ROW3
- D57 pad 1: /COL11 -> Net-(D57-K)
- D57 pad 2: Net-(D57-A) -> /ROW3
- D58 pad 1: /COL12 -> Net-(D58-K)
- D58 pad 2: Net-(D58-A) -> /ROW3
- D59 pad 1: /COL13 -> Net-(D59-K)
- D59 pad 2: Net-(D59-A) -> /ROW3
- D6 pad 1: /COL5 -> Net-(D6-K)
- D6 pad 2: Net-(D6-A) -> /ROW0
- D60 pad 1: /COL14 -> Net-(D60-K)
- D60 pad 2: Net-(D60-A) -> /ROW3
- D61 pad 1: /COL0 -> Net-(D61-K)
- D61 pad 2: Net-(D61-A) -> /ROW4
- D62 pad 1: /COL1 -> Net-(D62-K)
- D62 pad 2: Net-(D62-A) -> /ROW4
- D63 pad 1: /COL2 -> Net-(D63-K)
- D63 pad 2: Net-(D63-A) -> /ROW4
- D67 pad 1: /COL6 -> Net-(D67-K)
- D67 pad 2: Net-(D67-A) -> /ROW4
- D7 pad 1: /COL6 -> Net-(D7-K)
- D7 pad 2: Net-(D7-A) -> /ROW0
- D70 pad 1: /COL9 -> Net-(D70-K)
- D70 pad 2: Net-(D70-A) -> /ROW4
- D71 pad 1: /COL10 -> Net-(D71-K)
- D71 pad 2: Net-(D71-A) -> /ROW4
- D72 pad 1: /COL11 -> Net-(D72-K)
- D72 pad 2: Net-(D72-A) -> /ROW4
- D73 pad 1: /COL12 -> Net-(D73-K)
- D73 pad 2: Net-(D73-A) -> /ROW4
- D74 pad 1: /COL13 -> Net-(D74-K)
- D74 pad 2: Net-(D74-A) -> /ROW4
- D75 pad 1: /COL14 -> Net-(D75-K)
- D75 pad 2: Net-(D75-A) -> /ROW4
- D8 pad 1: /COL7 -> Net-(D8-K)
- D8 pad 2: Net-(D8-A) -> /ROW0
- D9 pad 1: /COL8 -> Net-(D9-K)
- D9 pad 2: Net-(D9-A) -> /ROW0
- SW1 pad 1: /ROW0 -> Net-(D1-K)
- SW1 pad 2: Net-(D1-A) -> /COL0
- SW10 pad 1: /ROW0 -> Net-(D10-K)
- SW10 pad 2: Net-(D10-A) -> /COL9
- SW11 pad 1: /ROW0 -> Net-(D11-K)
- SW11 pad 2: Net-(D11-A) -> /COL10
- SW12 pad 1: /ROW0 -> Net-(D12-K)
- SW12 pad 2: Net-(D12-A) -> /COL11
- SW13 pad 1: /ROW0 -> Net-(D13-K)
- SW13 pad 2: Net-(D13-A) -> /COL12
- SW14 pad 1: /ROW0 -> Net-(D14-K)
- SW14 pad 2: Net-(D14-A) -> /COL13
- SW16 pad 1: /ROW1 -> Net-(D16-K)
- SW16 pad 2: Net-(D16-A) -> /COL0
- SW17 pad 1: /ROW1 -> Net-(D17-K)
- SW17 pad 2: Net-(D17-A) -> /COL1
- SW18 pad 1: /ROW1 -> Net-(D18-K)
- SW18 pad 2: Net-(D18-A) -> /COL2
- SW19 pad 1: /ROW1 -> Net-(D19-K)
- SW19 pad 2: Net-(D19-A) -> /COL3
- SW2 pad 1: /ROW0 -> Net-(D2-K)
- SW2 pad 2: Net-(D2-A) -> /COL1
- SW20 pad 1: /ROW1 -> Net-(D20-K)
- SW20 pad 2: Net-(D20-A) -> /COL4
- SW21 pad 1: /ROW1 -> Net-(D21-K)
- SW21 pad 2: Net-(D21-A) -> /COL5
- SW22 pad 1: /ROW1 -> Net-(D22-K)
- SW22 pad 2: Net-(D22-A) -> /COL6
- SW23 pad 1: /ROW1 -> Net-(D23-K)
- SW23 pad 2: Net-(D23-A) -> /COL7
- SW24 pad 1: /ROW1 -> Net-(D24-K)
- SW24 pad 2: Net-(D24-A) -> /COL8
- SW25 pad 1: /ROW1 -> Net-(D25-K)
- SW25 pad 2: Net-(D25-A) -> /COL9
- SW26 pad 1: /ROW1 -> Net-(D26-K)
- SW26 pad 2: Net-(D26-A) -> /COL10
- SW27 pad 1: /ROW1 -> Net-(D27-K)
- SW27 pad 2: Net-(D27-A) -> /COL11
- SW28 pad 1: /ROW1 -> Net-(D28-K)
- SW28 pad 2: Net-(D28-A) -> /COL12
- SW29 pad 1: /ROW1 -> Net-(D29-K)
- SW29 pad 2: Net-(D29-A) -> /COL13
- SW3 pad 1: /ROW0 -> Net-(D3-K)
- SW3 pad 2: Net-(D3-A) -> /COL2
- SW31 pad 1: /ROW2 -> Net-(D31-K)
- SW31 pad 2: Net-(D31-A) -> /COL0
- SW32 pad 1: /ROW2 -> Net-(D32-K)
- SW32 pad 2: Net-(D32-A) -> /COL1
- SW33 pad 1: /ROW2 -> Net-(D33-K)
- SW33 pad 2: Net-(D33-A) -> /COL2
- SW34 pad 1: /ROW2 -> Net-(D34-K)
- SW34 pad 2: Net-(D34-A) -> /COL3
- SW35 pad 1: /ROW2 -> Net-(D35-K)
- SW35 pad 2: Net-(D35-A) -> /COL4
- SW36 pad 1: /ROW2 -> Net-(D36-K)
- SW36 pad 2: Net-(D36-A) -> /COL5
- SW37 pad 1: /ROW2 -> Net-(D37-K)
- SW37 pad 2: Net-(D37-A) -> /COL6
- SW38 pad 1: /ROW2 -> Net-(D38-K)
- SW38 pad 2: Net-(D38-A) -> /COL7
- SW39 pad 1: /ROW2 -> Net-(D39-K)
- SW39 pad 2: Net-(D39-A) -> /COL8
- SW4 pad 1: /ROW0 -> Net-(D4-K)
- SW4 pad 2: Net-(D4-A) -> /COL3
- SW40 pad 1: /ROW2 -> Net-(D40-K)
- SW40 pad 2: Net-(D40-A) -> /COL9
- SW41 pad 1: /ROW2 -> Net-(D41-K)
- SW41 pad 2: Net-(D41-A) -> /COL10
- SW42 pad 1: /ROW2 -> Net-(D42-K)
- SW42 pad 2: Net-(D42-A) -> /COL11
- SW44 pad 1: /ROW2 -> Net-(D44-K)
- SW44 pad 2: Net-(D44-A) -> /COL13
- SW46 pad 1: /ROW3 -> Net-(D46-K)
- SW46 pad 2: Net-(D46-A) -> /COL0
- SW48 pad 1: /ROW3 -> Net-(D48-K)
- SW48 pad 2: Net-(D48-A) -> /COL2
- SW49 pad 1: /ROW3 -> Net-(D49-K)
- SW49 pad 2: Net-(D49-A) -> /COL3
- SW5 pad 1: /ROW0 -> Net-(D5-K)
- SW5 pad 2: Net-(D5-A) -> /COL4
- SW50 pad 1: /ROW3 -> Net-(D50-K)
- SW50 pad 2: Net-(D50-A) -> /COL4
- SW51 pad 1: /ROW3 -> Net-(D51-K)
- SW51 pad 2: Net-(D51-A) -> /COL5
- SW52 pad 1: /ROW3 -> Net-(D52-K)
- SW52 pad 2: Net-(D52-A) -> /COL6
- SW53 pad 1: /ROW3 -> Net-(D53-K)
- SW53 pad 2: Net-(D53-A) -> /COL7
- SW54 pad 1: /ROW3 -> Net-(D54-K)
- SW54 pad 2: Net-(D54-A) -> /COL8
- SW55 pad 1: /ROW3 -> Net-(D55-K)
- SW55 pad 2: Net-(D55-A) -> /COL9
- SW56 pad 1: /ROW3 -> Net-(D56-K)
- SW56 pad 2: Net-(D56-A) -> /COL10
- SW57 pad 1: /ROW3 -> Net-(D57-K)
- SW57 pad 2: Net-(D57-A) -> /COL11
- SW58 pad 1: /ROW3 -> Net-(D58-K)
- SW58 pad 2: Net-(D58-A) -> /COL12
- SW59 pad 1: /ROW3 -> Net-(D59-K)
- SW59 pad 2: Net-(D59-A) -> /COL13
- SW6 pad 1: /ROW0 -> Net-(D6-K)
- SW6 pad 2: Net-(D6-A) -> /COL5
- SW60 pad 1: /ROW3 -> Net-(D60-K)
- SW60 pad 2: Net-(D60-A) -> /COL14
- SW61 pad 1: /ROW4 -> Net-(D61-K)
- SW61 pad 2: Net-(D61-A) -> /COL0
- SW62 pad 1: /ROW4 -> Net-(D62-K)
- SW62 pad 2: Net-(D62-A) -> /COL1
- SW63 pad 1: /ROW4 -> Net-(D63-K)
- SW63 pad 2: Net-(D63-A) -> /COL2
- SW67 pad 1: /ROW4 -> Net-(D67-K)
- SW67 pad 2: Net-(D67-A) -> /COL6
- SW7 pad 1: /ROW0 -> Net-(D7-K)
- SW7 pad 2: Net-(D7-A) -> /COL6
- SW70 pad 1: /ROW4 -> Net-(D70-K)
- SW70 pad 2: Net-(D70-A) -> /COL9
- SW71 pad 1: /ROW4 -> Net-(D71-K)
- SW71 pad 2: Net-(D71-A) -> /COL10
- SW72 pad 1: /ROW4 -> Net-(D72-K)
- SW72 pad 2: Net-(D72-A) -> /COL11
- SW73 pad 1: /ROW4 -> Net-(D73-K)
- SW73 pad 2: Net-(D73-A) -> /COL12
- SW74 pad 1: /ROW4 -> Net-(D74-K)
- SW74 pad 2: Net-(D74-A) -> /COL13
- SW75 pad 1: /ROW4 -> Net-(D75-K)
- SW75 pad 2: Net-(D75-A) -> /COL14
- SW8 pad 1: /ROW0 -> Net-(D8-K)
- SW8 pad 2: Net-(D8-A) -> /COL7
- SW9 pad 1: /ROW0 -> Net-(D9-K)
- SW9 pad 2: Net-(D9-A) -> /COL8
Routing:
- net /COL12: track 104.1 -> 557.8 mm, vias 0 -> 2
- net /COL13: track 109.7 -> 562.5 mm, vias 0 -> 2
- net /COL14: track 28.6 -> 478.5 mm, vias 0 -> 2
- net /COL10: track 113.5 -> 521.2 mm, vias 0 -> 2
- net /COL11: track 113.5 -> 518.3 mm, vias 0 -> 2
- net /COL9: track 113.5 -> 517.3 mm, vias 0 -> 2
- net /COL2: track 106.3 -> 493.9 mm, vias 0 -> 2
- net /COL1: track 96.4 -> 483.5 mm, vias 0 -> 2
- net /COL0: track 96.4 -> 482.1 mm, vias 0 -> 2
- net /COL5: track 80.4 -> 454.4 mm, vias 0 -> 2
- net /COL4: track 80.4 -> 453.3 mm, vias 0 -> 2
- net /COL3: track 80.4 -> 452.1 mm, vias 0 -> 2
- net /COL8: track 80.4 -> 445.0 mm, vias 0 -> 2
- net /COL7: track 80.4 -> 443.6 mm, vias 0 -> 2
- net /COL6: track 101.6 -> 463.4 mm, vias 0 -> 2
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Other:
- board text added: "A"
- board text added: "rev."
