File: hzk65_controller.kicad_sch (KiCad schematic)
At the start: 1 part

Commit message: Update gpios
Connections:
- net COL0: now also A1.19 (GPIO14); no longer A1.7 (GPIO5)
- net COL1: now also A1.17 (GPIO13); no longer A1.9 (GPIO6)
- net COL10: now also A1.2 (GPIO1); no longer A1.20 (GPIO15)
- net COL11: now also A1.1 (GPIO0); no longer A1.21 (GPIO16)
- net COL12: now also A1.24 (GPIO18); no longer A1.22 (GPIO17)
- net COL13: now also A1.22 (GPIO17); no longer A1.24 (GPIO18)
- net COL14: now also A1.21 (GPIO16); no longer A1.25 (GPIO19)
- net COL2: now also A1.16 (GPIO12); no longer A1.10 (GPIO7)
- net COL3: now also A1.14 (GPIO10); no longer A1.11 (GPIO8)
- net COL5: now also A1.11 (GPIO8); no longer A1.14 (GPIO10)
- net COL6: now also A1.9 (GPIO6); no longer A1.15 (GPIO11)
- net COL7: now also A1.7 (GPIO5); no longer A1.16 (GPIO12)
- net COL8: now also A1.6 (GPIO4); no longer A1.17 (GPIO13)
- net COL9: now also A1.4 (GPIO2); no longer A1.19 (GPIO14)
- net ROW0: now also A1.20 (GPIO15); no longer A1.1 (GPIO0)
- net ROW1: now also A1.15 (GPIO11); no longer A1.2 (GPIO1)
- net ROW2: now also A1.10 (GPIO7); no longer A1.4 (GPIO2)
- net ROW4: now also A1.25 (GPIO19); no longer A1.6 (GPIO4)
Changed lines of the file:
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@@
 	(hierarchical_label "ROW1"
 		(shape output)
+		(at 116.84 114.3 180)
+		(effects
+			(font
+				(size 1.27 1.27)
+			)
+			(justify right)
+		)
+	)
+	(hierarchical_label "COL14"
+		(shape input)
+		(at 162.56 88.9 0)
+		(effects
+			(font
+				(size 1.27 1.27)
+			)
+			(justify left)
+		)
+	)
+	(hierarchical_label "COL9"
+		(shape input)
+		(at 116.84 91.44 180)
+		(effects
+			(font
+				(size 1.27 1.27)
+			)
+			(justify right)
+		)
+	)
+	(hierarchical_label "ROW4"
+		(shape output)
+		(at 162.56 96.52 0)
+		(effects
+			(font
+				(size 1.27 1.27)
+			)
+			(justify left)
+		)
+	)
+	(hierarchical_label "COL3"
+		(shape input)
+		(at 116.84 111.76 180)
+		(effects
+			(font
+				(size 1.27 1.27)
+			)
+			(justify right)
+		)
+	)
+	(hierarchical_label "COL12"
+		(shape input)
+		(at 162.56 93.98 0)
+		(effects
+			(font
+				(size 1.27 1.27)
+			)
+			(justify left)
+		)
+	)
+	(hierarchical_label "COL6"
+		(shape input)
+		(at 116.84 101.6 180)
+		(effects
+			(font
+				(size 1.27 1.27)
+			)
+			(justify right)
+		)
+	)
+	(hierarchical_label "ROW2"
+		(shape output)
+		(at 116.84 104.14 180)
+		(effects
+			(font
+				(size 1.27 1.27)
+			)
+			(justify right)
+		)
+	)
+	(hierarchical_label "ROW0"
+		(shape output)
+		(at 116.84 124.46 180)
+		(effects
+			(font
+				(size 1.27 1.27)
+			)
+			(justify right)
+		)
+	)
+	(hierarchical_label "COL5"
+		(shape input)
+		(at 116.84 106.68 180)
+		(effects
+			(font
+				(size 1.27 1.27)
+			)
+			(justify right)
+		)
+	)
+	(hierarchical_label "COL13"
+		(shape input)
+		(at 162.56 91.44 0)
+		(effects
+			(font
+				(size 1.27 1.27)
+			)
+			(justify left)
+		)
+	)
+	(hierarchical_label "COL10"
+		(shape input)
 		(at 116.84 88.9 180)
 		(effects
@@
 		)
 	)
-	(hierarchical_label "COL14"
-		(shape input)
-		(at 162.56 96.52 0)
-		(effects
-			(font
-				(size 1.27 1.27)
-			)
-			(justify left)
-		)
-	)
-	(hierarchical_label "COL9"
+	(hierarchical_label "COL0"
 		(shape input)
 		(at 116.84 121.92 180)
@@
 		)
 	)
-	(hierarchical_label "ROW4"
-		(shape output)
+	(hierarchical_label "COL7"
+		(shape input)
+		(at 116.84 99.06 180)
+		(effects
+			(font
+				(size 1.27 1.27)
+			)
+			(justify right)
+		)
+	)
+	(hierarchical_label "COL2"
+		(shape input)
+		(at 116.84 116.84 180)
+		(effects
+			(font
+				(size 1.27 1.27)
+			)
+			(justify right)
+		)
+	)
+	(hierarchical_label "ROW3"
+		(shape output)
+		(at 116.84 93.98 180)
+		(effects
+			(font
+				(size 1.27 1.27)
+			)
+			(justify right)
+		)
+	)
+	(hierarchical_label "COL8"
+		(shape input)
 		(at 116.84 96.52 180)
 		(effects
@@
 		)
 	)
-	(hierarchical_label "COL3"
-		(shape input)
-		(at 116.84 106.68 180)
-		(effects
-			(font
-				(size 1.27 1.27)
-			)
-			(justify right)
-		)
-	)
-	(hierarchical_label "COL12"
-		(shape input)
-		(at 162.56 91.44 0)
-		(effects
-			(font
-				(size 1.27 1.27)
-			)
-			(justify left)
-		)
-	)
-	(hierarchical_label "COL6"
-		(shape input)
-		(at 116.84 114.3 180)
-		(effects
-			(font
-				(size 1.27 1.27)
-			)
-			(justify right)
-		)
-	)
-	(hierarchical_label "ROW2"
-		(shape output)
-		(at 116.84 91.44 180)
-		(effects
-			(font
-				(size 1.27 1.27)
-			)
-			(justify right)
-		)
-	)
-	(hierarchical_label "ROW0"
-		(shape output)
+	(hierarchical_label "COL1"
+		(shape input)
+		(at 116.84 119.38 180)
+		(effects
+			(font
+				(size 1.27 1.27)
+			)
+			(justify right)
+		)
+	)
+	(hierarchical_label "COL4"
+		(shape input)
+		(at 116.84 109.22 180)
+		(effects
+			(font
+				(size 1.27 1.27)
+			)
+			(justify right)
+		)
+	)
+	(hierarchical_label "COL11"
+		(shape input)
 		(at 116.84 86.36 180)
 		(effects
@@
 		)
 	)
-	(hierarchical_label "COL5"
-		(shape input)
-		(at 116.84 111.76 180)
-		(effects
-			(font
-				(size 1.27 1.27)
-			)
-			(justify right)
-		)
-	)
-	(hierarchical_label "COL13"
-		(shape input)
-		(at 162.56 93.98 0)
-		(effects
-			(font
-				(size 1.27 1.27)
-			)
-			(justify left)
-		)
-	)
-	(hierarchical_label "COL10"
-		(shape input)
-		(at 116.84 124.46 180)
-		(effects
-			(font
-				(size 1.27 1.27)
-			)
-			(justify right)
-		)
-	)
-	(hierarchical_label "COL0"
-		(shape input)
-		(at 116.84 99.06 180)
-		(effects
-			(font
-				(size 1.27 1.27)
-			)
-			(justify right)
-		)
-	)
-	(hierarchical_label "COL7"
-		(shape input)
-		(at 116.84 116.84 180)
-		(effects
-			(font
-				(size 1.27 1.27)
-			)
-			(justify right)
-		)
-	)
-	(hierarchical_label "COL2"
-		(shape input)
-		(at 116.84 104.14 180)
-		(effects
-			(font
-				(size 1.27 1.27)
-			)
-			(justify right)
-		)
-	)
-	(hierarchical_label "ROW3"
-		(shape output)
-		(at 116.84 93.98 180)
-		(effects
-			(font
-				(size 1.27 1.27)
-			)
-			(justify right)
-		)
-	)
-	(hierarchical_label "COL8"
-		(shape input)
-		(at 116.84 119.38 180)
-		(effects
-			(font
-				(size 1.27 1.27)
-			)
-			(justify right)
-		)
-	)
-	(hierarchical_label "COL1"
-		(shape input)
-		(at 116.84 101.6 180)
-		(effects
-			(font
-				(size 1.27 1.27)
-			)
-			(justify right)
-		)
-	)
-	(hierarchical_label "COL4"
-		(shape input)
-		(at 116.84 109.22 180)
-		(effects
-			(font
-				(size 1.27 1.27)
-			)
-			(justify right)
-		)
-	)
-	(hierarchical_label "COL11"
-		(shape input)
-		(at 162.56 88.9 0)
-		(effects
-			(font
-				(size 1.27 1.27)
-			)
-			(justify left)
-		)
-	)
