File: pcb/hzk65/hzk65_controller.kicad_sch (KiCad schematic)
At the start: 1 part

Commit message: Improve symmetrical routing
Connections:
- net COL10: now also A1.27 (GPIO21); no longer A1.2 (GPIO1)
- net COL11: now also A1.26 (GPIO20); no longer A1.1 (GPIO0)
- net COL5: now also A1.10 (GPIO7); no longer A1.11 (GPIO8)
- net COL6: now also A1.7 (GPIO5); no longer A1.9 (GPIO6)
- net COL7: now also A1.34 (GPIO28_ADC2); no longer A1.7 (GPIO5)
- net COL8: now also A1.32 (GPIO27_ADC1); no longer A1.6 (GPIO4)
- net COL9: now also A1.29 (GPIO22); no longer A1.4 (GPIO2)
- net ROW2: now also A1.9 (GPIO6); no longer A1.10 (GPIO7)
- net ROW3: now also A1.31 (GPIO26_ADC0); no longer A1.5 (GPIO3)
Changed lines of the file:
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@@
 	(paper "A4")
 	(no_connect
-		(at 162.56 104.14)
-	)
-	(no_connect
-		(at 162.56 119.38)
+		(at 116.84 93.98)
+	)
+	(no_connect
+		(at 116.84 88.9)
 	)
 	(no_connect
@@
 	)
 	(no_connect
-		(at 162.56 116.84)
-	)
-	(no_connect
-		(at 162.56 114.3)
+		(at 116.84 96.52)
+	)
+	(no_connect
+		(at 116.84 91.44)
 	)
 	(no_connect
@@
 	)
 	(no_connect
-		(at 162.56 101.6)
-	)
-	(no_connect
-		(at 162.56 99.06)
+		(at 116.84 106.68)
+	)
+	(no_connect
+		(at 116.84 86.36)
 	)
 	(no_connect
@@
 	(hierarchical_label "COL9"
 		(shape input)
-		(at 116.84 91.44 180)
-		(effects
-			(font
-				(size 1.27 1.27)
-			)
-			(justify right)
+		(at 162.56 104.14 0)
+		(effects
+			(font
+				(size 1.27 1.27)
+			)
+			(justify left)
 		)
 	)
@@
 	(hierarchical_label "COL6"
 		(shape input)
+		(at 116.84 99.06 180)
+		(effects
+			(font
+				(size 1.27 1.27)
+			)
+			(justify right)
+		)
+	)
+	(hierarchical_label "ROW2"
+		(shape output)
 		(at 116.84 101.6 180)
 		(effects
@@
 		)
 	)
-	(hierarchical_label "ROW2"
-		(shape output)
+	(hierarchical_label "ROW0"
+		(shape output)
+		(at 116.84 124.46 180)
+		(effects
+			(font
+				(size 1.27 1.27)
+			)
+			(justify right)
+		)
+	)
+	(hierarchical_label "COL5"
+		(shape input)
 		(at 116.84 104.14 180)
 		(effects
@@
 		)
 	)
-	(hierarchical_label "ROW0"
-		(shape output)
-		(at 116.84 124.46 180)
-		(effects
-			(font
-				(size 1.27 1.27)
-			)
-			(justify right)
-		)
-	)
-	(hierarchical_label "COL5"
-		(shape input)
-		(at 116.84 106.68 180)
-		(effects
-			(font
-				(size 1.27 1.27)
-			)
-			(justify right)
-		)
-	)
 	(hierarchical_label "COL13"
 		(shape input)
@@
 	(hierarchical_label "COL10"
 		(shape input)
-		(at 116.84 88.9 180)
-		(effects
-			(font
-				(size 1.27 1.27)
-			)
-			(justify right)
+		(at 162.56 101.6 0)
+		(effects
+			(font
+				(size 1.27 1.27)
+			)
+			(justify left)
 		)
 	)
@@
 	(hierarchical_label "COL7"
 		(shape input)
-		(at 116.84 99.06 180)
-		(effects
-			(font
-				(size 1.27 1.27)
-			)
-			(justify right)
+		(at 162.56 119.38 0)
+		(effects
+			(font
+				(size 1.27 1.27)
+			)
+			(justify left)
 		)
 	)
@@
 	(hierarchical_label "ROW3"
 		(shape output)
-		(at 116.84 93.98 180)
-		(effects
-			(font
-				(size 1.27 1.27)
-			)
-			(justify right)
+		(at 162.56 114.3 0)
+		(effects
+			(font
+				(size 1.27 1.27)
+			)
+			(justify left)
 		)
 	)
 	(hierarchical_label "COL8"
 		(shape input)
-		(at 116.84 96.52 180)
-		(effects
-			(font
-				(size 1.27 1.27)
-			)
-			(justify right)
+		(at 162.56 116.84 0)
+		(effects
+			(font
+				(size 1.27 1.27)
+			)
+			(justify left)
 		)
 	)
@@
 	(hierarchical_label "COL11"
 		(shape input)
-		(at 116.84 86.36 180)
-		(effects
-			(font
-				(size 1.27 1.27)
-			)
-			(justify right)
-		)
-	)
+		(at 162.56 99.06 0)
+		(effects
+			(font
+				(size 1.27 1.27)
+			)
+			(justify left)
+		)
+	)
