File: pcb/hzk65/hzk65.kicad_pcb (KiCad board)
At the start: 2 copper layers, 314.3 x 100 mm, 135 parts, among them SW1 SW_Push, SW10 SW_Push, SW11 SW_Push, SW12 SW_Push, SW13 SW_Push, SW14 SW_Push, SW16 SW_Push, SW17 SW_Push, SW18 SW_Push, SW19 SW_Push, SW2 SW_Push, SW20 SW_Push, SW21 SW_Push, SW22 SW_Push, SW23 SW_Push, SW24 SW_Push, SW25 SW_Push, SW26 SW_Push, SW27 SW_Push, SW28 SW_Push, SW29 SW_Push, SW3 SW_Push, SW31 SW_Push, SW32 SW_Push, SW33 SW_Push, SW34 SW_Push, SW35 SW_Push, SW36 SW_Push, SW37 SW_Push, SW38 SW_Push, SW39 SW_Push, SW4 SW_Push, SW40 SW_Push, SW41 SW_Push, SW42 SW_Push, SW44 SW_Push, SW46 SW_Push, SW48 SW_Push, SW49 SW_Push, SW5 SW_Push, SW50 SW_Push, SW51 SW_Push, SW52 SW_Push, SW53 SW_Push, SW54 SW_Push, SW55 SW_Push, SW56 SW_Push, SW57 SW_Push, SW58 SW_Push, SW59 SW_Push, SW6 SW_Push, SW60 SW_Push, SW61 SW_Push, SW62 SW_Push, SW63 SW_Push, SW67 SW_Push, SW7 SW_Push, SW70 SW_Push, SW71 SW_Push, SW72 SW_Push, SW73 SW_Push, SW74 SW_Push, SW75 SW_Push, SW8 SW_Push, SW9 SW_Push

Commit message: Improve symmetrical routing
Connections:
- A1 pad 1: /COL11 -> unconnected-(A1-GPIO0-Pad1)
- A1 pad 10: /ROW2 -> /COL5
- A1 pad 11: /COL5 -> unconnected-(A1-GPIO8-Pad11)
- A1 pad 2: /COL10 -> unconnected-(A1-GPIO1-Pad2)
- A1 pad 26: unconnected-(A1-GPIO20-Pad26) -> /COL11
- A1 pad 27: unconnected-(A1-GPIO21-Pad27) -> /COL10
- A1 pad 29: unconnected-(A1-GPIO22-Pad29) -> /COL9
- A1 pad 31: unconnected-(A1-GPIO26_ADC0-Pad31) -> /ROW3
- A1 pad 32: unconnected-(A1-GPIO27_ADC1-Pad32) -> /COL8
- A1 pad 34: unconnected-(A1-GPIO28_ADC2-Pad34) -> /COL7
- A1 pad 4: /COL9 -> unconnected-(A1-GPIO2-Pad4)
- A1 pad 5: /ROW3 -> unconnected-(A1-GPIO3-Pad5)
- A1 pad 6: /COL8 -> unconnected-(A1-GPIO4-Pad6)
- A1 pad 7: /COL7 -> /COL6
- A1 pad 9: /COL6 -> /ROW2
Routing:
- net /COL14: track 124.3 -> 423.2 mm, vias 4 -> 2
- net /COL13: track 225.3 -> 517.7 mm
- net /COL12: track 243.0 -> 516.8 mm
- net /COL11: track 277.8 -> 489.2 mm
- net /COL10: track 292.5 -> 491.8 mm
- net /COL9: track 304.7 -> 496.8 mm
- net /COL8: track 255.5 -> 433.4 mm
- net /COL7: track 270.8 -> 437.9 mm
- net /COL6: track 304.6 -> 457.7 mm
- net /COL5: track 314.9 -> 440.5 mm
- net /COL4: track 330.2 -> 433.5 mm
- net /COL3: track 343.0 -> 426.6 mm
- net /COL2: track 411.9 -> 465.8 mm
- net /COL1: track 414.2 -> 448.4 mm
- net /ROW2: track 352.5 -> 379.0 mm
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
Commit message: Improve routing for aesthetics
Parts:
- moved A1 0.36 mm to (346.2, 101.9)
- moved D12 0.36 mm to (271.8, 114.4)
- moved D13 0.36 mm to (290.8, 114.4)
- moved D14 0.36 mm to (319.4, 114.4)
- moved D19 0.36 mm to (128.9, 133.4)
- moved D20 0.36 mm to (148.0, 133.4)
- moved D26 0.36 mm to (262.3, 133.4)
- moved D27 0.36 mm to (281.3, 133.4)
- moved D28 0.36 mm to (300.4, 133.4)
- moved D5 0.36 mm to (138.4, 114.4)
- moved D59 0.36 mm to (333.7, 176.3)
- moved D6 0.36 mm to (157.5, 114.4)
- moved D71 0.36 mm to (271.8, 190.6)
- moved D72 0.36 mm to (290.8, 190.6)
- moved D73 0.36 mm to (314.6, 195.3)
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Routing:
- net /ROW4: track 427.2 -> 413.5 mm
- net /COL13: track 517.7 -> 503.9 mm
- net /COL12: track 516.8 -> 503.1 mm
- net /COL14: track 423.2 -> 421.4 mm
